File: hardware/wakeuplight rev1/_saved_wakeup light.sch (KiCad schematic (older format))
At the start: 20 parts, among them CON1 BARREL_JACK, CON2 Fog_Light, CON3 LED_Header, J1 Serial_Header, J2 1/8_MH, J3 1/8_MH, J4 1/8_MH, J5 1/8_MH, SW1 Rotary_Encoder, U1 Arduino_Pro_Mini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

Commit message: components placed
Schematics updated with mounting holes
components placed, need to wire them up
Parts:
- J2, J3, J4, J5: footprint Mounting_Holes:MountingHole_3mm -> wakeuplight rev1:2.5mm_MH
Changed lines of the file:
@@
 F 0 "J2" H 6500 1450 60  0000 C CNN
 F 1 "1/8_MH" H 6750 1100 60  0000 C CNN
-F 2 "Mounting_Holes:MountingHole_3mm" H 6550 1150 60  0001 C CNN
+F 2 "wakeuplight rev1:2.5mm_MH" H 6550 1150 60  0001 C CNN
 F 3 "" H 6550 1150 60  0000 C CNN
 	1    6550 1150
@@
 F 0 "J3" H 7000 1450 60  0000 C CNN
 F 1 "1/8_MH" H 7250 1100 60  0000 C CNN
-F 2 "Mounting_Holes:MountingHole_3mm" H 7050 1150 60  0001 C CNN
+F 2 "wakeuplight rev1:2.5mm_MH" H 7050 1150 60  0001 C CNN
 F 3 "" H 7050 1150 60  0000 C CNN
 	1    7050 1150
@@
 F 0 "J4" H 7500 1450 60  0000 C CNN
 F 1 "1/8_MH" H 7750 1100 60  0000 C CNN
-F 2 "Mounting_Holes:MountingHole_3mm" H 7550 1150 60  0001 C CNN
+F 2 "wakeuplight rev1:2.5mm_MH" H 7550 1150 60  0001 C CNN
 F 3 "" H 7550 1150 60  0000 C CNN
 	1    7550 1150
@@
 F 0 "J5" H 7950 1450 60  0000 C CNN
 F 1 "1/8_MH" H 8200 1100 60  0000 C CNN
-F 2 "Mounting_Holes:MountingHole_3mm" H 8000 1150 60  0001 C CNN
+F 2 "wakeuplight rev1:2.5mm_MH" H 8000 1150 60  0001 C CNN
 F 3 "" H 8000 1150 60  0000 C CNN
 	1    8000 1150
