File: hardware/wakeuplight rev1/wakeup light.sch (KiCad schematic (older format))
At the start: 20 parts, among them CON1 BARREL_JACK, CON2 Fog_Light, CON3 LED_Header, J1 Serial_Header, J2 1/8_MH, J3 1/8_MH, J4 1/8_MH, J5 1/8_MH, SW1 Rotary_Encoder, U1 Arduino_Pro_Mini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

Commit message: Completed layout
Wiring complete
Need to double check and send off to manufacture.
Parts:
- J2, J3, J4, J5: footprint Mounting_Holes:MountingHole_3mm -> wakeuplight rev1:2.5mm_MH
- renumbered CON1 to J6, CON3 to J7, CON2 to J8
Connections:
- net labels added: FogLightReturn
- wire segments 133 -> 137

Commit message: includes PDF schematics
For easier reading!
includes component values
Parts:
- C1, C2: value CP -> 100uF
- R1, R2, R3: value R -> 10k
Other:
- note added: "Time constant 1s"
Changed lines of the file:
@@
 P 4850 3700
 F 0 "R3" V 4930 3700 50  0000 C CNN
-F 1 "R" V 4850 3700 50  0000 C CNN
+F 1 "10k" V 4850 3700 50  0000 C CNN
 F 2 "Resistors_SMD:R_0603_HandSoldering" V 4780 3700 50  0001 C CNN
 F 3 "" H 4850 3700 50  0000 C CNN
@@
 P 5150 3950
 F 0 "C1" H 5175 4050 50  0000 L CNN
-F 1 "CP" H 5175 3850 50  0000 L CNN
+F 1 "100uF" H 5175 3850 50  0000 L CNN
 F 2 "wakeuplight rev1:Cap_Fat_1000uF_25V" H 5188 3800 50  0001 C CNN
 F 3 "" H 5150 3950 50  0000 C CNN
@@
 P 8800 1950
 F 0 "C2" H 8825 2050 50  0000 L CNN
-F 1 "CP" H 8825 1850 50  0000 L CNN
+F 1 "100uF" H 8825 1850 50  0000 L CNN
 F 2 "wakeuplight rev1:Cap_Fat_1000uF_25V" H 8838 1800 50  0001 C CNN
 F 3 "" H 8800 1950 50  0000 C CNN
@@
 P 2250 1650
 F 0 "R1" V 2330 1650 50  0000 C CNN
-F 1 "R" V 2250 1650 50  0000 C CNN
+F 1 "10k" V 2250 1650 50  0000 C CNN
 F 2 "Resistors_SMD:R_0603_HandSoldering" V 2180 1650 50  0001 C CNN
 F 3 "" H 2250 1650 50  0000 C CNN
@@
 P 2400 1650
 F 0 "R2" V 2480 1650 50  0000 C CNN
-F 1 "R" V 2400 1650 50  0000 C CNN
+F 1 "10k" V 2400 1650 50  0000 C CNN
 F 2 "Resistors_SMD:R_0603_HandSoldering" V 2330 1650 50  0001 C CNN
 F 3 "" H 2400 1650 50  0000 C CNN
@@
 Text Label 8800 4100 0    60   ~ 0
 FogLightReturn
+Text Notes 4200 3900 0    60   ~ 0
+Time constant 1s
 $EndSCHEMATC
